File: Kicad/ercf-ez-board.sch (KiCad schematic (older format))
At the start: 27 parts, among them J1 Conn_01x03_Male, J2 Conn_01x03_Male, J3 Conn_01x03_Male, J4 Conn_01x03_Male, J5 Screw_Terminal_01x02, J6 Conn_01x05_Male, J7 Conn_01x04_Male, J8 Conn_01x04_Male, U1 SeeeduinoXIAO, U2 L7805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

Commit message: Open 2nd jumper
Open the jumper for the second UART pin
Parts:
- JP7, JP9: footprint Jumper:SolderJumper-2_P1.3mm_Bridged_RoundedPad1.0x1.5mm -> Jumper:SolderJumper-2_P1.3mm_Open_RoundedPad1.0x1.5mm
Changed lines of the file:
@@
 F 0 "JP7" V 7950 2600 50  0000 C CNN
 F 1 "Jumper_NC_Small" H 7450 2600 50  0000 C CNN
-F 2 "Jumper:SolderJumper-2_P1.3mm_Bridged_RoundedPad1.0x1.5mm" H 7700 2500 50  0001 C CNN
+F 2 "Jumper:SolderJumper-2_P1.3mm_Open_RoundedPad1.0x1.5mm" H 7700 2500 50  0001 C CNN
 F 3 "~" H 7700 2500 50  0001 C CNN
 	1    7700 2500
@@
 F 0 "JP9" V 7950 5250 50  0000 C CNN
 F 1 "Jumper_NC_Small" H 7450 5250 50  0000 C CNN
-F 2 "Jumper:SolderJumper-2_P1.3mm_Bridged_RoundedPad1.0x1.5mm" H 7700 5150 50  0001 C CNN
+F 2 "Jumper:SolderJumper-2_P1.3mm_Open_RoundedPad1.0x1.5mm" H 7700 5150 50  0001 C CNN
 F 3 "~" H 7700 5150 50  0001 C CNN
 	1    7700 5150

Commit message: PCB v1.1
PCB v1.1:
- VCC for endstop, encoder and extra are now 3V3
- Fix gear stepper ground plane was not connected to GND
- Improve the tracks width for power and motors
Parts:
- removed JP10, JP8: Jumper_NC_Small, Jumper:SolderJumper-2_P1.3mm_Bridged_RoundedPad1.0x1.5mm, symbol Device:Jumper_NC_Small
- added JP7, JP9: Jumper_NO_Small, Jumper:SolderJumper-2_P1.3mm_Open_RoundedPad1.0x1.5mm, symbol Device:Jumper_NO_Small
- JP10: renamed from JP9; footprint Jumper:SolderJumper-2_P1.3mm_Open_RoundedPad1.0x1.5mm -> Jumper:SolderJumper-2_P1.3mm_Bridged_RoundedPad1.0x1.5mm
- JP8: renamed from JP7; footprint Jumper:SolderJumper-2_P1.3mm_Open_RoundedPad1.0x1.5mm -> Jumper:SolderJumper-2_P1.3mm_Bridged_RoundedPad1.0x1.5mm
Connections:
- net +3V3: now also J2.3 (Pin_3), J3.3 (Pin_3), J4.3 (Pin_3)
- net UART: now also JP7.2, JP9.2
- net at U3.JP1_4 (PDN/UART1): now also JP7.1; no longer JP8.2
- net at U3.JP1_5 (PDN/UART2): now also JP8.2
- net at U4.JP1_4 (PDN/UART1): now also JP9.1; no longer JP10.2
- net at U4.JP1_5 (PDN/UART2): now also JP10.2
- removed net VCC: J2.3 (Pin_3), J3.3 (Pin_3), J4.3 (Pin_3), U1.14 (5V)
- no-connect marks 11 -> 12
Other:
- moved on the sheet: JP10, JP8
Changed lines of the file:
@@
 Sheet 1 1
 Title "ERCF EZ BOARD"
-Date "31/05/2021"
-Rev "v1.0"
+Date "02/06/2021"
+Rev "v1.1"
 Comp "The ERCF fanclub"
 Comment1 "by Tircown"
@@
 	1    9850 1150
 	1    0    0    -1
-$EndComp
-$Comp
-L power:VCC #PWR01
-U 1 1 60B3D854
-P 3150 1350
-F 0 "#PWR01" H 3150 1200 50  0001 C CNN
-F 1 "VCC" V 3165 1478 50  0000 L CNN
-F 2 "" H 3150 1350 50  0001 C CNN
-F 3 "" H 3150 1350 50  0001 C CNN
-	1    3150 1350
-	0    1    1    0
 $EndComp
 $Comp
@@
 Text GLabel 3150 2250 2    50   Input ~ 0
 S-MIN
-$Comp
-L power:VCC #PWR04
-U 1 1 60B695DA
-P 5500 6400
-F 0 "#PWR04" H 5500 6250 50  0001 C CNN
-F 1 "VCC" V 5515 6527 50  0000 L CNN
-F 2 "" H 5500 6400 50  0001 C CNN
-F 3 "" H 5500 6400 50  0001 C CNN
-	1    5500 6400
-	0    -1   -1   0
-$EndComp
 Wire Wire Line
 	5350 4700 5800 4700
@@
 	1    0    0    -1
 $EndComp
-$Comp
-L Device:Jumper_NC_Small JP7
+Wire Wire Line
+	8150 2200 7700 2200
+Wire Wire Line
+	7700 2200 7700 2400
+Wire Wire Line
+	8150 2300 7800 2300
+Wire Wire Line
+	7800 2300 7800 2400
+Text GLabel 7800 5450 3    50   Input ~ 0
+UART
+Wire Wire Line
+	7700 5250 7700 5350
+Wire Wire Line
+	7700 5350 7800 5350
+Wire Wire Line
+	7800 5250 7800 5350
+Wire Wire Line
+	7800 5350 7800 5450
+Connection ~ 7800 5350
+Wire Wire Line
+	7700 4850 7700 5050
+Wire Wire Line
+	7800 4950 7800 5050
+Wire Wire Line
+	8150 4850 7700 4850
+Wire Wire Line
+	8150 4950 7800 4950
+$Comp
+L power:+3V3 #PWR0101
+U 1 1 60B7B4E3
+P 5500 6400
+F 0 "#PWR0101" H 5500 6250 50  0001 C CNN
+F 1 "+3V3" V 5515 6528 50  0000 L CNN
+F 2 "" H 5500 6400 50  0001 C CNN
+F 3 "" H 5500 6400 50  0001 C CNN
+	1    5500 6400
+	0    -1   -1   0
+$EndComp
+NoConn ~ 3150 1350
+$Comp
+L Device:Jumper_NC_Small JP10
+U 1 1 60B880EF
+P 7800 5150
+F 0 "JP10" V 7950 5000 50  0000 C CNN
+F 1 "Jumper_NC_Small" H 7550 5050 50  0000 C CNN
+F 2 "Jumper:SolderJumper-2_P1.3mm_Bridged_RoundedPad1.0x1.5mm" H 7800 5150 50  0001 C CNN
+F 3 "~" H 7800 5150 50  0001 C CNN
+	1    7800 5150
+	0    -1   -1   0
+$EndComp
+$Comp
+L Device:Jumper_NO_Small JP9
+U 1 1 60B8EB85
+P 7700 5150
+F 0 "JP9" V 7450 4950 50  0000 L CNN
+F 1 "Jumper_NO_Small" H 7950 5050 50  0000 C CNN
+F 2 "Jumper:SolderJumper-2_P1.3mm_Open_RoundedPad1.0x1.5mm" H 7700 5150 50  0001 C CNN
+F 3 "~" H 7700 5150 50  0001 C CNN
+	1    7700 5150
+	0    1    1    0
+$EndComp
+$Comp
+L Device:Jumper_NC_Small JP8
 U 1 1 60B6220C
-P 7700 2500
-F 0 "JP7" V 7950 2600 50  0000 C CNN
-F 1 "Jumper_NC_Small" H 7450 2600 50  0000 C CNN
-F 2 "Jumper:SolderJumper-2_P1.3mm_Open_RoundedPad1.0x1.5mm" H 7700 2500 50  0001 C CNN
-F 3 "~" H 7700 2500 50  0001 C CNN
-	1    7700 2500
-	0    -1   -1   0
-$EndComp
-$Comp
-L Device:Jumper_NC_Small JP8
-U 1 1 60B6E600
 P 7800 2500
 F 0 "JP8" V 7950 2400 50  0000 C CNN
@@
 	0    -1   -1   0
 $EndComp
-Wire Wire Line
-	8150 2200 7700 2200
-Wire Wire Line
-	7700 2200 7700 2400
-Wire Wire Line
-	8150 2300 7800 2300
-Wire Wire Line
-	7800 2300 7800 2400
-Text GLabel 7800 5450 3    50   Input ~ 0
-UART
-Wire Wire Line
-	7700 5250 7700 5350
-Wire Wire Line
-	7700 5350 7800 5350
-Wire Wire Line
-	7800 5250 7800 5350
-Wire Wire Line
-	7800 5350 7800 5450
-Connection ~ 7800 5350
-$Comp
-L Device:Jumper_NC_Small JP9
-U 1 1 60B880EF
-P 7700 5150
-F 0 "JP9" V 7950 5250 50  0000 C CNN
-F 1 "Jumper_NC_Small" H 7450 5250 50  0000 C CNN
-F 2 "Jumper:SolderJumper-2_P1.3mm_Open_RoundedPad1.0x1.5mm" H 7700 5150 50  0001 C CNN
-F 3 "~" H 7700 5150 50  0001 C CNN
-	1    7700 5150
-	0    -1   -1   0
-$EndComp
-$Comp
-L Device:Jumper_NC_Small JP10
-U 1 1 60B880F5
-P 7800 5150
-F 0 "JP10" V 7950 5050 50  0000 C CNN
-F 1 "Jumper_NC_Small" H 7550 5050 50  0000 C CNN
-F 2 "Jumper:SolderJumper-2_P1.3mm_Bridged_RoundedPad1.0x1.5mm" H 7800 5150 50  0001 C CNN
-F 3 "~" H 7800 5150 50  0001 C CNN
-	1    7800 5150
-	0    -1   -1   0
-$EndComp
-Wire Wire Line
-	7700 4850 7700 5050
-Wire Wire Line
-	7800 4950 7800 5050
-Wire Wire Line
-	8150 4850 7700 4850
-Wire Wire Line
-	8150 4950 7800 4950
+$Comp
+L Device:Jumper_NO_Small JP7
+U 1 1 60B87691
+P 7700 2500
+F 0 "JP7" V 7500 2300 50  0000 L CNN
+F 1 "Jumper_NO_Small" H 7950 2400 50  0000 C CNN
+F 2 "Jumper:SolderJumper-2_P1.3mm_Open_RoundedPad1.0x1.5mm" H 7700 2500 50  0001 C CNN
+F 3 "~" H 7700 2500 50  0001 C CNN
+	1    7700 2500
+	0    1    1    0
+$EndComp
 $EndSCHEMATC
