File: Kicad/ercf-easy-brd.sch (KiCad schematic (older format))
At the start: 27 parts, among them J1 Conn_01x03_Male, J2 Conn_01x03_Male, J3 Conn_01x03_Male, J4 Conn_01x03_Male, J5 Screw_Terminal_01x02, J6 Conn_01x05_Male, J7 Conn_01x04_Male, J8 Conn_01x04_Male, U1 SeeeduinoXIAO, U2 L7805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

Commit message: Rename project
Rename project from ercf-ez-board to ercf-easy-brd to avoid confusion: it is not a TH3D product.
Parts:
- J5: footprint ercf-ez-board:TerminalBlock_bornier-2_P5.08mm_2 -> ercf-easy-brd:TerminalBlock_bornier-2_P5.08mm_2
- J6: footprint ercf-ez-board:PinHeader_1x05_P2.54mm_Vertical_2 -> ercf-easy-brd:PinHeader_1x05_P2.54mm_Vertical_2
- U1: footprint ercf-ez-board:SeeeduinoXIAO-MODULE14P -> ercf-easy-brd:SeeeduinoXIAO-MODULE14P; symbol ercf-ez-board:SeeeduinoXIAO -> ercf-easy-brd:SeeeduinoXIAO
- U3, U4: footprint ercf-ez-board:MODULE_TMC2209_SILENTSTEPSTICK -> ercf-easy-brd:MODULE_TMC2209_SILENTSTEPSTICK; symbol ercf-ez-board:TMC2209_SILENTSTEPSTICK -> ercf-easy-brd:TMC2209_SILENTSTEPSTICK
Changed lines of the file:
@@
 encoding utf-8
 Sheet 1 1
-Title "ERCF EZ BOARD"
+Title "ERCF EASY BRD"
 Date "02/06/2021"
 Rev "v1.1"
@@
 $EndDescr
 $Comp
-L ercf-ez-board:SeeeduinoXIAO U1
+L ercf-easy-brd:SeeeduinoXIAO U1
 U 1 1 60ACCCFB
 P 2350 1800
 F 0 "U1" H 2325 861 50  0000 C CNN
 F 1 "SeeeduinoXIAO" H 2325 770 50  0000 C CNN
-F 2 "ercf-ez-board:SeeeduinoXIAO-MODULE14P" H 2000 2000 50  0001 C CNN
+F 2 "ercf-easy-brd:SeeeduinoXIAO-MODULE14P" H 2000 2000 50  0001 C CNN
 F 3 "" H 2000 2000 50  0001 C CNN
 	1    2350 1800
@@
 	8150 2500 8050 2500
 $Comp
-L ercf-ez-board:TMC2209_SILENTSTEPSTICK U3
+L ercf-easy-brd:TMC2209_SILENTSTEPSTICK U3
 U 1 1 60AD171B
 P 8850 1900
 F 0 "U3" H 8850 2767 50  0000 C CNN
 F 1 "TMC2209_SILENTSTEPSTICK" H 8850 2676 50  0000 C CNN
-F 2 "ercf-ez-board:MODULE_TMC2209_SILENTSTEPSTICK" H 8850 1900 50  0001 L BNN
+F 2 "ercf-easy-brd:MODULE_TMC2209_SILENTSTEPSTICK" H 8850 1900 50  0001 L BNN
 F 3 "" H 8850 1900 50  0001 L BNN
 F 4 "v11" H 8850 1900 50  0001 L BNN "PARTREV"
@@
 	8150 5150 8050 5150
 $Comp
-L ercf-ez-board:TMC2209_SILENTSTEPSTICK U4
+L ercf-easy-brd:TMC2209_SILENTSTEPSTICK U4
 U 1 1 60AF166A
 P 8850 4550
 F 0 "U4" H 8850 5417 50  0000 C CNN
 F 1 "TMC2209_SILENTSTEPSTICK" H 8850 5326 50  0000 C CNN
-F 2 "ercf-ez-board:MODULE_TMC2209_SILENTSTEPSTICK" H 8850 4550 50  0001 L BNN
+F 2 "ercf-easy-brd:MODULE_TMC2209_SILENTSTEPSTICK" H 8850 4550 50  0001 L BNN
 F 3 "" H 8850 4550 50  0001 L BNN
 F 4 "v11" H 8850 4550 50  0001 L BNN "PARTREV"
@@
 F 0 "J5" V 5750 1150 50  0000 R CNN
 F 1 "Screw_Terminal_01x02" V 5650 1500 50  0000 R CNN
-F 2 "ercf-ez-board:TerminalBlock_bornier-2_P5.08mm_2" H 5500 1150 50  0001 C CNN
+F 2 "ercf-easy-brd:TerminalBlock_bornier-2_P5.08mm_2" H 5500 1150 50  0001 C CNN
 F 3 "~" H 5500 1150 50  0001 C CNN
 	1    5500 1150
@@
 F 0 "J6" H 6200 6300 50  0000 C CNN
 F 1 "Conn_01x05_Male" H 6200 6200 50  0000 C CNN
-F 2 "ercf-ez-board:PinHeader_1x05_P2.54mm_Vertical_2" H 6200 5850 50  0001 C CNN
+F 2 "ercf-easy-brd:PinHeader_1x05_P2.54mm_Vertical_2" H 6200 5850 50  0001 C CNN
 F 3 "~" H 6200 5850 50  0001 C CNN
 	1    6200 5850
